Commit message: roll the wheels

File: PHASE_3/simple_robot.urdf (robot description, URDF)
Before this commit: robot two_wheel_robot, 4 links, 3 joints
Links:
- link left_wheel: geometry collision origin rpy=1.5707 0 0; visual cylinder length=0.02 radius=0.05

Commit message: roll the wheels

File: PHASE_3/simple_robot.urdf (robot description, URDF)
Before this commit: robot two_wheel_robot, 4 links, 3 joints
Links:
- link base_link: mass None -> 3.0
- link caster_wheel: mass None -> 0.1
- link left_wheel: mass None -> 0.3; geometry collision cylinder length=0.02 radius=0.05; visual cylinder length=0.02 radius=0.05
- link right_wheel: mass None -> 0.3

Commit message: 3-3 fin

File: PHASE_3/simple_robot.urdf (robot description, URDF)
Before this commit: robot two_wheel_robot, 4 links, 3 joints
Links:
- link caster_wheel: geometry collision sphere radius=0.05; visual sphere radius=0.05
Joints:
- joint left_wheel_joint: origin xyz=0 0.1 -0.05 -> xyz=0.1 0.1 -0.05
- joint right_wheel_joint: origin xyz=0 -0.1 -0.05 -> xyz=0.1 -0.1 -0.05
