Commit message: update

File: PHASE_3/maze_escaper_3_9/urdf/wheeled_robot.urdf (robot description, URDF)
Before this commit: robot wheeled_robot, 4 links, 3 joints
Links:
- added link camera_link, mass 0.05; collision box size=0.04 0.04 0.04; visual box size=0.04 0.04 0.04
- added link caster_wheel_front, mass 0.05; collision sphere radius=0.025; visual sphere radius=0.025
- added link lidar_link, mass 0.1; collision cylinder length=0.04 radius=0.05; visual cylinder length=0.04 radius=0.05
Joints:
- added joint camera_joint: type fixed, parent base_link, child camera_link, origin xyz=0.13 0 0.05 rpy=0 0 0
- added joint caster_joint_front: type fixed, parent base_link, child caster_wheel_front, origin xyz=0.1 0 -0.075 rpy=0 0 0
- added joint lidar_joint: type fixed, parent base_link, child lidar_link, origin xyz=0 0 0.13 rpy=0 0 0
